File: board_faboboard/PCB/FaboBoard.sch (EAGLE design)
At the start: 42 parts, among them U1 FT232RL, U2 ATMEGA328P-AU, U7 TEMT6000, U8 LMV358, U9 MIC9.7MM, Y1 16MHz

Commit message: update FaboBoard
Parts:
- added U$3: (no value), Gclue:LOGO_OSHW-S
- LED1, LED2: device Gclue:LED0603 -> Gclue:LED-EIA0603
- U$2: device Gclue:LOGO_FABKURA -> Gclue:LOGO_GCLUE
Other:
- note removed: "fabkura.org"
Changed lines of the file:
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@@
 <part name="R1" library="Gclue" deviceset="RESISTOR" device="0603" value="1k"/>
 <part name="R2" library="Gclue" deviceset="RESISTOR" device="0603" value="1k"/>
-<part name="LED1" library="Gclue" deviceset="LED" device="0603" value="Red"/>
-<part name="LED2" library="Gclue" deviceset="LED" device="0603" value="Green"/>
+<part name="LED1" library="Gclue" deviceset="LED" device="-EIA0603" value="Red"/>
+<part name="LED2" library="Gclue" deviceset="LED" device="-EIA0603" value="Green"/>
 <part name="SUPPLY3" library="Gclue" deviceset="5V" device=""/>
 <part name="SUPPLY4" library="Gclue" deviceset="5V" device=""/>
@@
 <part name="C11" library="Gclue" deviceset="CAPACITOR" device="0603" value="0.1uF"/>
 <part name="U$1" library="Gclue" deviceset="A4L-LOC" device=""/>
-<part name="U$2" library="Gclue" deviceset="LOGO_FABKURA" device=""/>
+<part name="U$2" library="Gclue" deviceset="LOGO_GCLUE" device=""/>
+<part name="U$3" library="Gclue" deviceset="LOGO_OSHW" device="-S"/>
 </parts>
 <sheets>
@@
 <text x="81.28" y="7.62" size="1.6764" layer="94">Released under the Creative Commons Attribution Share-Alike 3.0 License</text>
 <text x="81.28" y="5.08" size="1.6764" layer="94">http://creativecommons.org/licenses/by-sa/3.0</text>
-<text x="199.644" y="5.334" size="1.6764" layer="94" font="vector">fabkura.org</text>
 <text x="217.17" y="15.24" size="1.9304" layer="94">PicoBoard compatible</text>
 <text x="247.65" y="5.08" size="1.9304" layer="94">v 0.1</text>
@@
 <instance part="C11" gate="G$1" x="246.38" y="154.94"/>
 <instance part="U$1" gate="G$1" x="0" y="0"/>
-<instance part="U$2" gate="G$1" x="207.264" y="11.43"/>
+<instance part="U$2" gate="G$1" x="210.82" y="20.32"/>
+<instance part="U$3" gate="G$1" x="167.64" y="7.62"/>
 </instances>
 <busses>
