File: brick_analog_angle/PCB/angle_brick.sch (EAGLE design)
At the start: 2 parts, among them J1 3PIN, U1 ANGLE

Commit message: Add data for elecrow
Parts:
- J2: value 3PIN -> (none)
- renumbered J1 to J2
Changed lines of the file:
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@@
 <layer number="97" name="Info" color="7" fill="1" visible="yes" active="yes"/>
 <layer number="98" name="Guide" color="6" fill="1" visible="yes" active="yes"/>
+<layer number="99" name="SpiceOrder" color="7" fill="1" visible="no" active="no"/>
 <layer number="100" name="Muster" color="7" fill="1" visible="no" active="no"/>
 <layer number="101" name="Patch_Top" color="12" fill="4" visible="no" active="yes"/>
@@
 <layer number="111" name="LPC17xx" color="7" fill="1" visible="yes" active="yes"/>
 <layer number="112" name="tSilk" color="7" fill="1" visible="yes" active="yes"/>
+<layer number="113" name="IDFDebug" color="4" fill="1" visible="yes" active="yes"/>
 <layer number="116" name="Patch_BOT" color="9" fill="4" visible="no" active="yes"/>
 <layer number="121" name="_tsilk" color="7" fill="1" visible="no" active="yes"/>
@@
 <parts>
 <part name="U$1" library="gclue" deviceset="A4L-LOC" device=""/>
-<part name="J1" library="gclue" deviceset="BRICK_3PIN" device="" value="3PIN"/>
 <part name="U1" library="gclue" deviceset="ROTARYENCORDER_BRICK" device="" value="ANGLE"/>
+<part name="J2" library="gclue" deviceset="BRICK_3PIN" device=""/>
 </parts>
 <sheets>
@@
 <instances>
 <instance part="U$1" gate="G$1" x="0" y="0"/>
-<instance part="J1" gate="G$1" x="91.44" y="88.9" smashed="yes">
-<attribute name="NAME" x="86.36" y="97.028" size="1.778" layer="95"/>
-</instance>
 <instance part="U1" gate="G$1" x="154.94" y="88.9" smashed="yes" rot="R180">
 <attribute name="NAME" x="149.86" y="97.028" size="1.778" layer="95"/>
 <attribute name="VALUE" x="152.4" y="78.74" size="1.778" layer="96"/>
 </instance>
+<instance part="J2" gate="G$1" x="91.44" y="88.9"/>
 </instances>
 <busses>
@@
 <net name="N$1" class="0">
 <segment>
-<pinref part="J1" gate="G$1" pin="I/O"/>
 <pinref part="U1" gate="G$1" pin="6"/>
 <wire x1="99.06" y1="93.98" x2="144.78" y2="93.98" width="0.1524" layer="91"/>
+<pinref part="J2" gate="G$1" pin="I/O"/>
 </segment>
 </net>
 <net name="VCC" class="0">
 <segment>
-<pinref part="J1" gate="G$1" pin="VCC"/>
 <wire x1="99.06" y1="88.9" x2="116.84" y2="88.9" width="0.1524" layer="91"/>
 <wire x1="116.84" y1="88.9" x2="127" y2="83.82" width="0.1524" layer="91"/>
 <pinref part="U1" gate="G$1" pin="2"/>
 <wire x1="127" y1="83.82" x2="144.78" y2="83.82" width="0.1524" layer="91"/>
+<pinref part="J2" gate="G$1" pin="VCC"/>
 </segment>
 </net>
 <net name="GND" class="0">
 <segment>
-<pinref part="J1" gate="G$1" pin="GND"/>
 <wire x1="99.06" y1="83.82" x2="116.84" y2="83.82" width="0.1524" layer="91"/>
 <wire x1="116.84" y1="83.82" x2="127" y2="88.9" width="0.1524" layer="91"/>
 <pinref part="U1" gate="G$1" pin="4"/>
 <wire x1="127" y1="88.9" x2="144.78" y2="88.9" width="0.1524" layer="91"/>
+<pinref part="J2" gate="G$1" pin="GND"/>
 </segment>
 </net>
