File: beacon_bluegiga/ble113/square/akabeacon_square_type2.sch (EAGLE design)
At the start: 9 parts

Commit message: Update rev.beta
Other:
- moved on the sheet: TC1
Changed lines of the file:
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@@
 <instance part="GND9" gate="1" x="144.78" y="116.84" rot="R90"/>
 <instance part="P+4" gate="G$1" x="96.52" y="116.84" rot="R90"/>
-<instance part="TC1" gate="A" x="119.38" y="121.92"/>
+<instance part="TC1" gate="A" x="116.84" y="121.92"/>
 <instance part="U$3" gate="G$1" x="20.32" y="83.82"/>
 </instances>
@@
 </segment>
 <segment>
-<wire x1="142.24" y1="116.84" x2="127" y2="116.84" width="0.1524" layer="91"/>
+<wire x1="142.24" y1="116.84" x2="124.46" y2="116.84" width="0.1524" layer="91"/>
 <pinref part="GND9" gate="1" pin="GND"/>
 <pinref part="TC1" gate="A" pin="1"/>
@@
 </segment>
 <segment>
-<wire x1="96.52" y1="116.84" x2="111.76" y2="116.84" width="0.1524" layer="91"/>
+<wire x1="96.52" y1="116.84" x2="109.22" y2="116.84" width="0.1524" layer="91"/>
 <pinref part="P+4" gate="G$1" pin="3.3V"/>
 <pinref part="TC1" gate="A" pin="2"/>
@@
 </segment>
 <segment>
-<wire x1="142.24" y1="119.38" x2="127" y2="119.38" width="0.1524" layer="91"/>
+<wire x1="142.24" y1="119.38" x2="124.46" y2="119.38" width="0.1524" layer="91"/>
 <label x="142.24" y="119.38" size="1.778" layer="95" rot="R180"/>
 <pinref part="TC1" gate="A" pin="3"/>
@@
 </segment>
 <segment>
-<wire x1="95.25" y1="119.38" x2="111.76" y2="119.38" width="0.1524" layer="91"/>
+<wire x1="95.25" y1="119.38" x2="109.22" y2="119.38" width="0.1524" layer="91"/>
 <label x="96.52" y="119.38" size="1.778" layer="95"/>
 <pinref part="TC1" gate="A" pin="4"/>
@@
 </segment>
 <segment>
-<wire x1="142.24" y1="121.92" x2="127" y2="121.92" width="0.1524" layer="91"/>
+<wire x1="142.24" y1="121.92" x2="124.46" y2="121.92" width="0.1524" layer="91"/>
 <label x="139.7" y="121.92" size="1.778" layer="95" rot="R180"/>
 <pinref part="TC1" gate="A" pin="5"/>
@@
 </segment>
 <segment>
-<wire x1="111.76" y1="121.92" x2="96.52" y2="121.92" width="0.1524" layer="91"/>
+<wire x1="109.22" y1="121.92" x2="96.52" y2="121.92" width="0.1524" layer="91"/>
 <label x="96.52" y="121.92" size="1.778" layer="95"/>
 <pinref part="TC1" gate="A" pin="6"/>
@@
 </segment>
 <segment>
-<wire x1="127" y1="124.46" x2="142.24" y2="124.46" width="0.1524" layer="91"/>
+<wire x1="124.46" y1="124.46" x2="142.24" y2="124.46" width="0.1524" layer="91"/>
 <label x="142.24" y="124.46" size="1.778" layer="95"/>
 <pinref part="TC1" gate="A" pin="7"/>

Commit message: Update BLE113
Parts:
- removed C3: 100uF, SparkFun-Capacitors:10UF-6.3V-20%(1206)
- TC1: value TC2050-IDC-NL -> TC2050-IDC; device TagConnect:TC2050-IDC-NL -> TagConnect:TC2050-IDC
Connections:
- net 3.3V: no longer C3.2
- net GND: no longer C3.1
Changed lines of the file:
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@@
 <part name="U$5" library="gclue" deviceset="BLE113" device=""/>
 <part name="GND4" library="SparkFun" deviceset="GND" device=""/>
-<part name="C3" library="SparkFun-Capacitors" deviceset="10UF-6.3V-20%(1206)" device="" value="100uF"/>
 <part name="U$1" library="gclue" deviceset="A4L-LOC" device=""/>
 <part name="R1" library="GClue-Resistors" deviceset="RESISTOR" device="0603" value="4.7K"/>
@@
 <part name="GND9" library="SparkFun" deviceset="GND" device=""/>
 <part name="P+4" library="SparkFun" deviceset="3.3V" device=""/>
-<part name="TC1" library="TagConnect" deviceset="TC2050-IDC" device="-NL" value=""/>
+<part name="TC1" library="TagConnect" deviceset="TC2050-IDC" device="" value="TC2050-IDC"/>
 <part name="U$3" library="GClue-Beacon" deviceset="SQUARE-TYPE2-TC2050" device=""/>
 </parts>
@@
 <instance part="U$5" gate="G$1" x="106.68" y="58.42"/>
 <instance part="GND4" gate="1" x="137.16" y="33.02"/>
-<instance part="C3" gate="G$1" x="60.96" y="68.58" rot="R90"/>
 <instance part="U$1" gate="G$1" x="0" y="0"/>
 <instance part="R1" gate="G$1" x="38.1" y="111.76"/>
@@
 <pinref part="GND1" gate="1" pin="GND"/>
 <wire x1="50.8" y1="81.28" x2="50.8" y2="76.2" width="0.1524" layer="91"/>
-<wire x1="50.8" y1="76.2" x2="50.8" y2="68.58" width="0.1524" layer="91"/>
-<wire x1="50.8" y1="68.58" x2="50.8" y2="66.04" width="0.1524" layer="91"/>
+<wire x1="50.8" y1="76.2" x2="50.8" y2="66.04" width="0.1524" layer="91"/>
 <wire x1="55.88" y1="76.2" x2="50.8" y2="76.2" width="0.1524" layer="91"/>
-<wire x1="50.8" y1="68.58" x2="55.88" y2="68.58" width="0.1524" layer="91"/>
-<pinref part="C3" gate="G$1" pin="1"/>
 <pinref part="C1" gate="G$1" pin="1"/>
 <wire x1="35.56" y1="81.28" x2="27.94" y2="81.28" width="0.1524" layer="91"/>
@@
 <wire x1="71.12" y1="86.36" x2="71.12" y2="88.9" width="0.1524" layer="91"/>
 <wire x1="63.5" y1="76.2" x2="71.12" y2="76.2" width="0.1524" layer="91"/>
-<wire x1="63.5" y1="68.58" x2="71.12" y2="68.58" width="0.1524" layer="91"/>
-<wire x1="71.12" y1="68.58" x2="71.12" y2="76.2" width="0.1524" layer="91"/>
-<pinref part="C3" gate="G$1" pin="2"/>
 <pinref part="C1" gate="G$1" pin="2"/>
 <wire x1="35.56" y1="86.36" x2="27.94" y2="86.36" width="0.1524" layer="91"/>
