File: 504_outin_chirimen/PCB/504_outin_chirimen.brd (EAGLE design)
At the start: 48 x 80 mm, 19 parts

Commit message: Update chirimen
Parts:
- removed I2C_0, I2C_2: (no value), FaBo-Template:FABO_BRICK_I2C_S04B-PASK-2
- removed SERIAL_0, SERIAL_3: (no value), FaBo-Template:FABO_BRICK_SERIAL_S04B-PASK-2
- removed U$22: (no value), FaBo-etc:LOGO_OSHW_T_MS_BOTTOM
- added GPIO6_A1: (no value), FaBo-Template:FABO_BRICK_3PIN_HEADER
- added I2C0_1, I2C0_2, I2C2_1, I2C2_2: (no value), FaBo-Template:FABO_BRICK_I2C_CONNECTOR_I_SILK
- added SERIAL0, SERIAL3: (no value), FaBo-Template:FABO_BRICK_SERIAL_CONNECTOR_I_SILK
- added U$3: (no value), FaBo-etc:LOGO_OSHW_T_M
- moved R3 25.7 mm to (44.5, 74.9)
- moved R4 25.7 mm to (44.5, 76.2)
- moved R1 25.7 mm to (44.5, 72.4)
- moved R2 25.7 mm to (44.5, 73.7)
- moved Q1 24.1 mm to (41.7, 69.1)
- moved R5 19.2 mm to (3.81, 72.4)
- moved R7 19.2 mm to (3.81, 74.9)
- moved R8 19.2 mm to (3.81, 76.2)
- moved R6 19.2 mm to (3.81, 73.7)
- moved Q2 13.6 mm to (6.35, 69.6)
- moved U$10 2.03 mm to (24.1, 13.5)
- moved ADC0_IN 1.27 mm to (24.1, 22.9)
- moved PWM0 1.27 mm to (20.3, 22.9)
Connections:
- new net GPIO6_A1: GPIO6_A1.I/O, U$2.CN2_15
- net 5V: now also GPIO6_A1.VCC, I2C0_1.VCC, I2C0_2.VCC, I2C2_1.VCC, I2C2_2.VCC, SERIAL0.VCC, SERIAL3.VCC; no longer I2C_0.VCC, I2C_2.VCC, SERIAL_0.VCC, SERIAL_3.VCC
- net GND: now also GPIO6_A1.GND, I2C0_1.GND, I2C0_2.GND, I2C2_1.GND, I2C2_2.GND, SERIAL0.GND, SERIAL3.GND, U$2.CN1_15; no longer I2C_0.GND, I2C_2.GND, SERIAL_0.GND, SERIAL_3.GND
- net RX0: now also SERIAL3.RX; no longer SERIAL_3.RX
- net RX3: now also SERIAL0.RX; no longer SERIAL_0.RX
- net SCL0: now also I2C0_1.SCL, I2C0_2.SCL; no longer I2C_2.SCL
- net SCL2: now also I2C2_1.SCL, I2C2_2.SCL; no longer I2C_0.SCL
- net SDA0: now also I2C0_1.SDA, I2C0_2.SDA; no longer I2C_2.SDA
- net SDA2: now also I2C2_1.SDA, I2C2_2.SDA; no longer I2C_0.SDA
- net TX0: now also SERIAL3.TX; no longer SERIAL_3.TX
- net TX3: now also SERIAL0.TX; no longer SERIAL_0.TX
Routing:
- net GND: track 0.00 -> 263.6 mm, vias 0 -> 17
- net 5V: track 0.00 -> 182.2 mm, vias 0 -> 2
- net 3V3: track 0.00 -> 98.2 mm, vias 0 -> 3
- net UART0_RX: track 0.00 -> 84.9 mm, vias 0 -> 1
- net UART3_TX: track 0.00 -> 84.8 mm, vias 0 -> 4
- net UART3_RX: track 0.00 -> 82.3 mm, vias 0 -> 4
- net UART0_TX: track 0.00 -> 81.0 mm, vias 0 -> 2
- net SDA2: track 0.00 -> 73.3 mm
- net SCL0: track 0.00 -> 66.4 mm
- net SDA0: track 0.00 -> 65.5 mm, vias 0 -> 1
- net SCL2: track 0.00 -> 63.2 mm
- net RX3: track 0.00 -> 54.2 mm
- net TX0: track 0.00 -> 34.1 mm, vias 0 -> 2
- net TX3: track 0.00 -> 33.6 mm
- net GPIO6_A1: track 0.00 -> 32.1 mm
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- added copper zone on layer 1, net GND
- added copper zone on layer 16, net GND
Other:
- outline, holes or cut-outs redrawn
- board text added: "I2C0"
- board text added: "I2C2"
- board text added: "Made In Japan"
- board text added: "Rev Beta1"
- board text added: "SERIAL0"
- board text added: "SERIAL3"

Commit message: Update chairmen
Parts:
- removed ADC0_IN, GPIO6_A1: (no value), FaBo-Template:FABO_BRICK_3PIN_HEADER
- added ADC0, GPIO6: (no value), FaBo-Template:FABO_BRICK_3PIN_HEADER
- added C1: 0.1uf, FaBo-Capacitor:0402
- added C2: 1uf, FaBo-Capacitor:0402
- added D1, D2, D3, D4, D5, D6, D7, D8: (no value), FaBo-Template:FABO_BRICK_3PIN_B03B-PASK-1_SILK
- added IC: TI-ADS7828, FaBo-ADC:TI-ADS7828
- added R10, R9: 4.7K, FaBo-Resistors:0402
- moved U$3 59.7 mm to (43.4, 62.5)
- moved PWM0 16.2 mm to (24.1, 7.11), turned to 0 degrees
- moved U$10 16.0 mm to (13.7, 1.27)
- moved R1 6.28 mm to (42.9, 66.3)
- moved R5 6.23 mm to (5.08, 66.3)
- moved R2 6.04 mm to (42.9, 67.8)
- moved R6 5.98 mm to (5.08, 67.8)
- moved R3 5.79 mm to (42.9, 69.3)
- moved R7 5.73 mm to (5.08, 69.3)
- moved R4 5.55 mm to (42.9, 70.9)
- moved R8 5.48 mm to (5.08, 70.9)
- moved Q1 4.64 mm to (42.4, 73.7)
- moved Q2 4.13 mm to (5.59, 73.7)
- moved I2C2_1 1.27 mm to (31.8, 54.6)
- moved I2C2_2 1.27 mm to (16.5, 54.6)
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Connections:
- new net CH0: D1.I/O, IC.1
- new net CH1: D2.I/O, IC.2
- new net CH2: D3.I/O, IC.3
- new net CH3: D4.I/O, IC.4
- new net CH4: D5.I/O, IC.5
- new net CH5: D6.I/O, IC.6
- new net CH6: D7.I/O, IC.7
- new net CH7: D8.I/O, IC.8
- new net N$3: C1.P$1, IC.10
- net 5V: now also ADC0.VCC, C2.P$1, D1.VCC, D2.VCC, D3.VCC, D4.VCC, D5.VCC, D6.VCC, D7.VCC, D8.VCC, GPIO6.VCC, IC.16, R10.P$2, R9.P$2; no longer ADC0_IN.VCC, GPIO6_A1.VCC
- net ADC0_IN: now also ADC0.I/O; no longer ADC0_IN.I/O
- net GND: now also ADC0.GND, C1.P$2, C2.P$2, D1.GND, D2.GND, D3.GND, D4.GND, D5.GND, D6.GND, D7.GND, D8.GND, GPIO6.GND, IC.11, IC.12, IC.13, IC.9; no longer ADC0_IN.GND, GPIO6_A1.GND
- net GPIO6_A1: now also GPIO6.I/O; no longer GPIO6_A1.I/O
- net SCL0: now also IC.14, R9.P$1
- net SDA0: now also IC.15, R10.P$1
Routing:
- net N$3: track 0.00 -> 75.9 mm
- net CH7: track 0.00 -> 70.7 mm, vias 0 -> 1
- net CH5: track 0.00 -> 61.1 mm, vias 0 -> 1
- net CH3: track 0.00 -> 58.4 mm, vias 0 -> 2
- net CH6: track 0.00 -> 56.1 mm, vias 0 -> 2
- net GND: track 263.6 -> 319.6 mm, vias 17 -> 46
- net 5V: track 182.2 -> 237.7 mm
- net CH2: track 0.00 -> 47.5 mm, vias 0 -> 2
- net CH4: track 0.00 -> 44.9 mm, vias 0 -> 2
- net CH1: track 0.00 -> 44.1 mm, vias 0 -> 2
- net SDA0: track 65.5 -> 104.2 mm, vias 1 -> 0
- net CH0: track 0.00 -> 38.5 mm, vias 0 -> 1
- net TX0: track 34.1 -> 68.4 mm, vias 2 -> 1
- net PWM0: track 18.5 -> 37.6 mm, vias 0 -> 1
- net SCL0: track 66.4 -> 81.3 mm, vias 0 -> 4
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Other:
- board text removed: "Made In Japan"

Commit message: Update beacon
Parts:
- removed I2C0_1, I2C0_2, I2C2_1, I2C2_2: (no value), FaBo-Template:FABO_BRICK_I2C_CONNECTOR_I_SILK
- removed SERIAL0, SERIAL3: (no value), FaBo-Template:FABO_BRICK_SERIAL_CONNECTOR_I_SILK
- added I2C1, I2C2, I2C3, I2C4: (no value), FaBo-Template:FABO_BRICK_I2C_B04B-PASK-1_SILK
- added J1, J2: (no value), FaBo-Template:FABO_BRICK_SERIAL_S04B-PASK-2_SILK
Connections:
- net 5V: now also I2C1.VCC, I2C2.VCC, I2C3.VCC, I2C4.VCC, J1.VCC, J2.VCC; no longer I2C0_1.VCC, I2C0_2.VCC, I2C2_1.VCC, I2C2_2.VCC, SERIAL0.VCC, SERIAL3.VCC
- net GND: now also I2C1.GND, I2C2.GND, I2C3.GND, I2C4.GND, J1.GND, J2.GND; no longer I2C0_1.GND, I2C0_2.GND, I2C2_1.GND, I2C2_2.GND, SERIAL0.GND, SERIAL3.GND
- net RX0: now also J1.RX; no longer SERIAL3.RX
- net RX3: now also J2.RX; no longer SERIAL0.RX
- net SCL0: now also I2C2.SCL, I2C4.SCL; no longer I2C0_1.SCL, I2C0_2.SCL
- net SCL2: now also I2C1.SCL, I2C3.SCL; no longer I2C2_1.SCL, I2C2_2.SCL
- net SDA0: now also I2C2.SDA, I2C4.SDA; no longer I2C0_1.SDA, I2C0_2.SDA
- net SDA2: now also I2C1.SDA, I2C3.SDA; no longer I2C2_1.SDA, I2C2_2.SDA
- net TX0: now also J1.TX; no longer SERIAL3.TX
- net TX3: now also J2.TX; no longer SERIAL0.TX
Routing:
- net SCL0: track 81.3 -> 144.4 mm, vias 4 -> 1
- net N$3: track 75.9 -> 15.2 mm, vias 0 -> 2
- net RX3: track 67.9 -> 20.5 mm, vias 1 -> 0
- net TX0: track 68.4 -> 25.8 mm, vias 1 -> 0
- net CH5: track 61.1 -> 40.0 mm, vias 1 -> 0
- net RX0: track 34.5 -> 15.1 mm
- net SCL2: track 65.9 -> 81.3 mm
- net GND: track 319.6 -> 334.8 mm, vias 46 -> 34
- net UART0_RX: track 93.1 -> 104.4 mm, vias 2 -> 3
- net 3V3: track 100.2 -> 110.4 mm, vias 2 -> 1
- net CH4: track 44.9 -> 34.9 mm
- net SDA0: track 104.2 -> 114.1 mm, vias 0 -> 2
- net CH0: track 38.5 -> 30.5 mm, vias 1 -> 2
- net CH1: track 44.1 -> 36.2 mm, vias 2 -> 1
- net GPIO6_A1: track 36.8 -> 29.2 mm
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