File: 0119_reflector/PCB/119_reflector.brd (EAGLE design)
At the start: 25.4 x 33 mm, 6 parts

Commit message: 9Aix_106A_Update,reflectorUpdate
Other:
- board text added: "Reflector"
- board text added: "Rev.1.0.0 B"
- board text added: "TOP"
- board text removed: "Refrector"
- board text removed: "Rev.1.0.0"
Changed lines of the file:
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@@
 <?xml version="1.0" encoding="utf-8"?>
 <!DOCTYPE eagle SYSTEM "eagle.dtd">
-<eagle version="8.2.2">
+<eagle version="8.7.1">
 <drawing>
 <settings>
 <setting alwaysvectorfont="no"/>
+<setting keepoldvectorfont="yes"/>
 <setting verticaltext="up"/>
 </settings>
@@
 <text x="22.86" y="12.065" size="0.8128" layer="21" font="vector" ratio="12" rot="R90" align="top-center">MADE IN JAPAN</text>
 <text x="3.175" y="12.7" size="2.54" layer="21" font="vector" ratio="12" rot="R90" align="bottom-center">#119</text>
-<text x="5.08" y="8.255" size="1.27" layer="21" font="vector" ratio="12" rot="R90">Refrector</text>
-<text x="6.985" y="8.255" size="1.016" layer="21" font="vector" ratio="12" rot="R90">Rev.1.0.0</text>
+<text x="5.08" y="8.255" size="1.27" layer="21" font="vector" ratio="12" rot="R90">Reflector</text>
+<text x="6.985" y="8.255" size="1.016" layer="21" font="vector" ratio="12" rot="R90">Rev.1.0.0 B</text>
+<text x="14.605" y="25.4" size="1.27" layer="21" font="vector" ratio="12" rot="R180">TOP</text>
 </plain>
 <attributes>
@@
 <param name="dpMaxLengthDifference" value="10mm"/>
 <param name="dpGapFactor" value="2.5"/>
-<param name="checkGrid" value="0"/>
 <param name="checkAngle" value="0"/>
 <param name="checkFont" value="1"/>
 <param name="checkRestrict" value="0"/>
+<param name="checkStop" value="0"/>
+<param name="checkValues" value="0"/>
 <param name="useDiameter" value="13"/>
 <param name="maxErrors" value="50"/>

Commit message: 0119_reflector　ロゴ修正、リファイン
Parts:
- removed U$4: (no value), FaBo-etc:LOGO_FABO_MS
- added LOGO1: (no value), component:LOGO_FABO_M
Routing:
- net I/O: track 23.7 -> 20.5 mm
- net N$1: track 12.6 -> 10.3 mm
- net VCC: track 12.7 -> 11.8 mm
Other:
- board text added: "Designed in Aizu"
- board text added: "Rev.1.0.1"
- board text removed: "MADE IN JAPAN"
- board text removed: "Rev.1.0.0 B"

Commit message: #0119 reflector プルアップ抵抗を103から102へ変更。
Parts:
- R2: value 10K -> 1K
Changed lines of the file:
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@@
 <?xml version="1.0" encoding="utf-8"?>
 <!DOCTYPE eagle SYSTEM "eagle.dtd">
-<eagle version="9.6.2">
+<eagle version="9.6.0">
 <drawing>
 <settings>
@@
 <attribute name="VALUE" x="14.24" y="20.665" size="0.8128" layer="27" font="vector" ratio="12" rot="R270" align="top-left"/>
 </element>
-<element name="R2" library="FaBo-Resistors" package="AXL-REGULAR" value="10K" x="10.795" y="18.415" smashed="yes" rot="R90">
+<element name="R2" library="FaBo-Resistors" package="AXL-REGULAR" value="1K" x="10.795" y="18.415" smashed="yes" rot="R90">
 <attribute name="NAME" x="10.795" y="16.165" size="0.8128" layer="25" font="vector" ratio="15" rot="R90" align="center-left"/>
 <attribute name="VALUE" x="11.795" y="16.165" size="0.8128" layer="27" font="vector" ratio="12" rot="R90" align="top-left"/>
