File: 0225_gps/pcb/225_gps.sch (EAGLE design)
At the start: 16 parts

Commit message: Update .
Parts:
- removed C3: 0.1uF, FaBo-Capacitor:CAPACITOR-0603
- removed C4: 1uF, FaBo-Capacitor:CAPACITOR-0603
- added R4, R5: 10K, FaBo-Resistors:RESISTOR-0603
- added TP3, TP4: (no value), FaBo-Supply:TP-15
- R1, R2: value 4.7k -> 2.2k
Connections:
- removed net +3V3: C1.2, C3.2, C4.2, IC2.VOUT, R1.2, R2.2, U$4.VCC
- new net 1V8: C1.2, IC2.VOUT, R1.2, R2.2, U$4.VCC(1V8)
- new net N$2: R4.2, U$4.RTS
- new net N$4: TP3.1, U$4.FORCE_ON
- new net N$5: R5.2, RESET.3, RESET.4, TP4.1
- net GND: now also R4.1, R5.1; no longer C3.1, C4.1, RESET.3, RESET.4, U$4.FORCE_ON

Commit message: Update gps.
Connections:
- removed net N$3: IC3.VREF1
- net 1V8: now also IC3.VREF1
Changed lines of the file:
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@@
 <part name="TP4" library="FaBo-Supply" deviceset="TP" device="-15"/>
 <part name="R5" library="FaBo-Resistors" deviceset="RESISTOR" device="-0603" value="10K"/>
+<part name="1V5" library="FaBo-Supply" deviceset="1V8" device=""/>
 </parts>
 <sheets>
@@
 <instance part="TP4" gate="G$1" x="149.86" y="81.28"/>
 <instance part="R5" gate="G$1" x="137.16" y="66.04" rot="R90"/>
+<instance part="1V5" gate="G$1" x="50.8" y="76.2"/>
 </instances>
 <busses>
@@
 </segment>
 </net>
-<net name="N$3" class="0">
-<segment>
-<wire x1="58.42" y1="55.88" x2="53.34" y2="55.88" width="0.1524" layer="91"/>
-<pinref part="IC3" gate="G$1" pin="VREF1"/>
-</segment>
-</net>
 <net name="RESET" class="0">
 <segment>
@@
 <wire x1="182.88" y1="152.4" x2="182.88" y2="160.02" width="0.1524" layer="91"/>
 </segment>
-</net>
+<segment>
+<wire x1="58.42" y1="55.88" x2="50.8" y2="55.88" width="0.1524" layer="91"/>
+<pinref part="IC3" gate="G$1" pin="VREF1"/>
+<wire x1="50.8" y1="55.88" x2="50.8" y2="76.2" width="0.1524" layer="91"/>
+<pinref part="1V5" gate="G$1" pin="1V8"/>
+</segment>
+</net>

Commit message: #225 gps ロゴ修正、リファイン
Parts:
- removed U$3: (no value), FaBo-etc:LOGO_FABO-M
- added LOGO1: (no value), component:LOGO_FABO-M
Other:
- note added: "1.0.0.Beta2"
- note removed: "1.0.0.Beta"
