File: 0230_color/pcb/230_color.sch (EAGLE design)
At the start: 16 parts

Commit message: #230 color ロゴ修正、リファイン
Parts:
- removed C4: 1uF, FaBo-Capacitor:CAPACITOR-0603
- removed U$3: (no value), FaBo-etc:LOGO_FABO-M
- removed U$5: ROHM-BH1749, FaBo-Mems:ROHM-BH1749
- added C3: 0.1uF, component:CAPACITOR-0603
- added IC1: (no value), component:BH1749NUC
- added LOGO1: (no value), component:LOGO_FABO-M
- added TP3: (no value), component:TP-15
- C1, C2: device FaBo-Capacitor:CAPACITOR-0603 -> component:CAPACITOR-0603
- R1, R2, R3, R4: device FaBo-Resistors:RESISTOR-0603 -> component:RESISTOR-0603
Connections:
- removed net ADDRESS: R4.2, SJ1.2, U$5.ADDR
- new net ADDR: IC1.ADDR, R4.2, SJ1.2
- new net INT: IC1.INT, TP3.1
- net 3V3: now also C3.2, IC1.VCC; no longer C4.1, U$5.VCC
- net GND: now also C3.1, IC1.GND@3, IC1.GND@9, IC1.TEST; no longer C4.2, U$5.GND, U$5.INT, U$5.TEST
- net SCL: now also IC1.SCL; no longer U$5.SCL
- net SDA: now also IC1.SDA; no longer U$5.SDA
Other:
- note added: "1.0.1 Beta"
- note added: "I2C address Default: 0x38 SJ1 short: 0x39"
- note removed: "1.0.5"
- moved on the sheet: IC2
