File: 0235_temperature/pcb/235_temperature.sch (EAGLE design)
At the start: 14 parts

Commit message: #235 temperature ロゴ修正、リファイン
Parts:
- removed ADT7420: ANALOGDEVICES-ADT7420, FaBo-Environment:ANALOGDEVICES-ADT7420
- removed C2, C4: 0.1uF, FaBo-Capacitor:CAPACITOR-0603
- removed IC2: (no value), FaBo-Supply:LP2985-33DBV
- removed IC3: (no value), FaBo-LevelTranslator:PCA9306GM
- removed R2: 4.7k, FaBo-Resistors:RESISTOR-0603
- removed R3: 200k, FaBo-Resistors:RESISTOR-0603
- removed R4: 10k, FaBo-Resistors:RESISTOR-0603
- removed SJ1: OPEN, FaBo-etc:SMD-JUMPER-2
- removed U$3: (no value), FaBo-etc:LOGO_FABO-M
- added IC1: (no value), component:ADT7420
- added JP1, JP2: open, component:JUMPER-2_SMD
- added LOGO1: (no value), component:LOGO_FABO-M
- added TP1, TP2: (no value), component:TP-15
- C1: value 1uF -> (none); device FaBo-Capacitor:CAPACITOR-0603 -> component:CAPACITOR-0603
- R1: value 4.7k -> 10k; device FaBo-Resistors:RESISTOR-0603 -> component:RESISTOR_ARRAY_4
Connections:
- removed net 3V3: ADT7420.VDD, C1.2, C4.1, IC2.VOUT, IC3.VREF1, R1.2, R2.2, SJ1.1
- removed net 5V: IC2.ON/OFF, IC2.VIN, J1.VCC, R3.2
- removed net ADDRESS: ADT7420.A0, R4.2, SJ1.2
- removed net N$1: C2.2, IC3.EN, IC3.VREF2, R3.1
- removed net SCL_HV: IC3.SCL2, J1.SCL
- removed net SDA_HV: IC3.SDA2, J1.SDA
- new net A0: IC1.A0, JP1.2, R1-A.2
- new net A1: IC1.A1, JP2.2, R1-B.2
- new net CT: IC1.CT, R1-D.2, TP2.1
- new net INT: IC1.INT, R1-C.2, TP1.1
- new net VCC: C1.2, IC1.VDD, J1.VCC, JP1.1, JP2.1, R1-C.1, R1-D.1
- net GND: now also IC1.EP, IC1.GND, R1-A.1, R1-B.1; no longer ADT7420.A1, ADT7420.GND, C2.1, C4.2, IC2.GND, IC3.GND, R4.1
- net SCL: now also IC1.SCL, J1.SCL; no longer ADT7420.SDA, IC3.SCL1, R1.1
- net SDA: now also IC1.SDA, J1.SDA; no longer ADT7420.SCL, IC3.SDA1, R2.1
Other:
- note added: "1.0.0 Beta"
- note removed: "1.0.5"
- moved on the sheet: C1, J1
