File: 0505_outin_kinomacreate/PCB/505_outin_kinoma.brd (EAGLE design)
At the start: 90 x 35 mm, 19 parts

Commit message: #505 outin_kinomacreate　ロゴ修正
Parts:
- removed U$3: (no value), FaBo-etc:LOGO_FABO_MS
- added LOGO1: (no value), component:LOGO_FABO_M
Other:
- board text added: "Designed in Aizu"
- board text removed: "MADE IN JAPAN"
