File: 0716_breakout_i2s/PCB/716_breakout_i2s.brd (EAGLE design)
At the start: 17.8 x 25.4 mm, 4 parts

Commit message: #716 breakout_i2s　ロゴ修正
Parts:
- U$2: device FaBo-etc:LOGO_FABO_MS_BOTTOM -> FaBo-Logo:LOGO_OSHW_M_BOTTOM
- U$3: device FaBo-etc:LOGO_OSHW_S_BOTTOM -> FaBo-Logo:LOGO_FABO_MS_BOTTOM
- moved U$2 5.08 mm to (9.53, 7.62)
- moved U$3 3.24 mm to (9.53, 12.1)
Other:
- board text added: "Designed in Aizu"
- board text removed: "MADE IN JAPAN"
