File: 0612_jetracer/PCB/612_jetracer_328_214.sch (EAGLE design)
At the start: 85 parts, among them IC2 JETSON_NANO_NOBORDER, IC3 MULTIPLEXERSMC74HC157A, M1 MOSFET-N_FDN335N, M2 MOSFET-N_FDN335N, M3 MOSFET-N_FDN335N, M4 MOSFET-N_FDN335N, M5 MOSFET-N_FDN335N, M6 MOSFET-N_FDN335N, Q1 MOSFET-N_FDN335N, Q2 MOSFET-N_FDN335N, X2 16MHz

Commit message: #612 JetRacer ファイルリネーム,シルク追加位置修正、GNDビア追加
Parts:
- R15, R21, R26, R30, R4, R6: value 10K -> 1K
Other:
- note added: "2021/9/7 Rev 2.0.14 ボディ装着のため、基板レイアウト変更"
Changed lines of the file:
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@@
 <part name="R17" library="FaBo-Resistors" deviceset="RESISTOR" device="-0603" value="47"/>
 <part name="R20" library="FaBo-Resistors" deviceset="RESISTOR" device="-0603" value="47"/>
-<part name="R4" library="FaBo-Resistors" deviceset="RESISTOR" device="-0603" value="10K"/>
-<part name="R6" library="FaBo-Resistors" deviceset="RESISTOR" device="-0603" value="10K"/>
+<part name="R4" library="FaBo-Resistors" deviceset="RESISTOR" device="-0603" value="1K"/>
+<part name="R6" library="FaBo-Resistors" deviceset="RESISTOR" device="-0603" value="1K"/>
 <part name="D3" library="Diode" library_urn="urn:adsk.eagle:library:16378169" deviceset="DIODE_" device="_SOD123G" package3d_urn="urn:adsk.eagle:package:9427058/2" technology="1N4148W-7-F" value="1N4148W"/>
 <part name="R27" library="FaBo-Resistors" deviceset="RESISTOR" device="-0603" value="4.7K"/>
@@
 <part name="GND8" library="FaBo-etc" deviceset="GND" device=""/>
 <part name="GND9" library="FaBo-etc" deviceset="GND" device=""/>
-<part name="R15" library="FaBo-Resistors" deviceset="RESISTOR" device="-0603" value="10K"/>
-<part name="R21" library="FaBo-Resistors" deviceset="RESISTOR" device="-0603" value="10K"/>
+<part name="R15" library="FaBo-Resistors" deviceset="RESISTOR" device="-0603" value="1K"/>
+<part name="R21" library="FaBo-Resistors" deviceset="RESISTOR" device="-0603" value="1K"/>
 <part name="D2" library="Diode" library_urn="urn:adsk.eagle:library:16378169" deviceset="DIODE_" device="_SOD123G" package3d_urn="urn:adsk.eagle:package:9427058/2" technology="1N4148W-7-F" value="1N4148W"/>
 <part name="R24" library="FaBo-Resistors" deviceset="RESISTOR" device="-0603" value="4.7K"/>
@@
 <part name="GND20" library="FaBo-etc" deviceset="GND" device=""/>
 <part name="GND26" library="FaBo-etc" deviceset="GND" device=""/>
-<part name="R26" library="FaBo-Resistors" deviceset="RESISTOR" device="-0603" value="10K"/>
-<part name="R30" library="FaBo-Resistors" deviceset="RESISTOR" device="-0603" value="10K"/>
+<part name="R26" library="FaBo-Resistors" deviceset="RESISTOR" device="-0603" value="1K"/>
+<part name="R30" library="FaBo-Resistors" deviceset="RESISTOR" device="-0603" value="1K"/>
 <part name="D4" library="Diode" library_urn="urn:adsk.eagle:library:16378169" deviceset="DIODE_" device="_SOD123G" package3d_urn="urn:adsk.eagle:package:9427058/2" technology="1N4148W-7-F" value="1N4148W"/>
 <part name="R31" library="FaBo-Resistors" deviceset="RESISTOR" device="-0603" value="4.7K"/>
@@
 <text x="544.83" y="431.8" size="3.81" layer="97">PWM Controller</text>
 <text x="557.53" y="373.38" size="1.778" layer="97">Address 0x40</text>
-<text x="492.76" y="147.32" size="3.81" layer="97">MULTIPLEXERS</text>
+<text x="472.44" y="181.61" size="3.81" layer="97">MULTIPLEXERS</text>
 <text x="896.62" y="97.79" size="1.778" layer="91" rot="MR0">D11</text>
 <text x="896.62" y="95.25" size="1.778" layer="91" rot="MR0">D12</text>
@@
 <text x="707.39" y="689.61" size="1.778" layer="94">SN74LVC1G17</text>
 <text x="1085.85" y="684.53" size="1.778" layer="94">SN74LVC1G17</text>
+<text x="830.58" y="472.44" size="6.4516" layer="94">2021/9/7 Rev 2.0.14 ボディ装着のため、基板レイアウト変更</text>
 </plain>
 <instances>

Commit message: #612 JetRacer RCのみ操縦のため電源経路変更
Parts:
- added C10: 1uF, FaBo-Capacitor:CAPACITOR-0603
- added C22: 4.7uF, FaBo-Capacitor:CAPACITOR-0603
- added C23: 0.01uF, FaBo-Capacitor:CAPACITOR-0603
- added D5: 1N4148W, Diode:DIODE_1N4148W-7-F_SOD123G
- added IC5: (no value), FaBo-Supply:LP2985-33DBV
Connections:
- new net N$47: C23.2, IC5.BYPASS
- new net N$48: C10.2, D5.C, IC5.ON/OFF, IC5.VIN
- new net RC_3V3: C22.2, IC5.VOUT, U$14.VCC, U$20.VCC, U$23.VCC
- net 3V3: no longer U$14.VCC, U$20.VCC, U$23.VCC
- net GND: now also C10.1, C22.1, C23.1, IC5.GND
- net VCC_RC: now also D5.A
Other:
- note added: "2.0.14"
- note added: "2021/9/8 Rev 2.0.14 ボディ装着のため、基板レイアウト変更,RC電源のみで走行可能"
- note added: "Analog 3V3"
- note added: "ESC"
- note added: "サーボ"
- note added: "受信機から入力"
- note removed: "2.0.13"
- note removed: "2021/9/7 Rev 2.0.14 ボディ装着のため、基板レイアウト変更"

Commit message: #612 JetRacer PCA9685 OEとボタンを追加
Parts:
- added R41: DNP, FaBo-Resistors:RESISTOR-0603
- added SW1: (no value), FaBo-Switch:TACT-SWITCH-SMD_KMR2
Connections:
- new net OE_PIN: IC1.ADC7, IC4.OE, R3.2
- net 3V3: now also R41.2
- net GND: now also SW1.1, SW1.2
- net N$7: now also IC1.ADC6, R41.1, SW1.3, SW1.4; no longer IC4.OE, R3.2
Changed lines of the file:
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@@
 <part name="GND77" library="FaBo-etc" deviceset="GND" device=""/>
 <part name="D5" library="Diode" library_urn="urn:adsk.eagle:library:16378169" deviceset="DIODE_" device="_SOD123G" package3d_urn="urn:adsk.eagle:package:9427058/2" technology="1N4148W-7-F" value="1N4148W"/>
+<part name="GND56" library="FaBo-Supply" deviceset="GND" device=""/>
+<part name="R41" library="FaBo-Resistors" deviceset="RESISTOR" device="-0603" value="DNP"/>
+<part name="3V6" library="FaBo-Supply" deviceset="3V3" device=""/>
+<part name="SW1" library="FaBo-Switch" deviceset="TACT-SWITCH" device="-SMD_KMR2"/>
 </parts>
 <sheets>
@@
 <attribute name="VALUE" x="209.55" y="730.25" size="1.778" layer="95" align="center"/>
 </instance>
+<instance part="GND56" gate="G$1" x="858.52" y="137.16" smashed="yes" rot="MR0">
+<attribute name="VALUE" x="861.314" y="132.08" size="1.778" layer="96" rot="MR0"/>
+</instance>
+<instance part="R41" gate="G$1" x="892.81" y="149.86" smashed="yes" rot="MR90">
+<attribute name="NAME" x="894.334" y="147.574" size="1.4224" layer="95" rot="MR90"/>
+<attribute name="VALUE" x="891.286" y="147.574" size="1.4224" layer="96" rot="MR90" align="top-left"/>
+</instance>
+<instance part="3V6" gate="G$1" x="892.81" y="176.53" smashed="yes" rot="MR0">
+<attribute name="VALUE" x="894.08" y="182.626" size="1.778" layer="96" rot="MR0"/>
+</instance>
+<instance part="SW1" gate="G$1" x="877.57" y="142.24" smashed="yes">
+<attribute name="NAME" x="877.57" y="147.574" size="1.27" layer="95" align="bottom-center"/>
+<attribute name="VALUE" x="877.57" y="138.43" size="1.27" layer="96" align="top-center"/>
+</instance>
 </instances>
 <busses>
@@
 <wire x1="276.86" y1="715.01" x2="276.86" y2="712.47" width="0.1524" layer="91"/>
 </segment>
+<segment>
+<wire x1="872.49" y1="139.7" x2="868.68" y2="139.7" width="0.1524" layer="91"/>
+<wire x1="868.68" y1="139.7" x2="868.68" y2="142.24" width="0.1524" layer="91"/>
+<wire x1="868.68" y1="142.24" x2="872.49" y2="142.24" width="0.1524" layer="91"/>
+<wire x1="868.68" y1="139.7" x2="858.52" y2="139.7" width="0.762" layer="91"/>
+<junction x="868.68" y="139.7"/>
+<pinref part="GND56" gate="G$1" pin="GND"/>
+<wire x1="858.52" y1="139.7" x2="858.52" y2="137.16" width="0.762" layer="91"/>
+<pinref part="SW1" gate="G$1" pin="1"/>
+<pinref part="SW1" gate="G$1" pin="2"/>
+</segment>
 </net>
 <net name="SDA" class="0">
@@
 <wire x1="619.76" y1="170.18" x2="622.3" y2="170.18" width="0.1524" layer="91"/>
 </segment>
-</net>
-<net name="N$7" class="0">
+<segment>
+<pinref part="3V6" gate="G$1" pin="3V3"/>
+<pinref part="R41" gate="G$1" pin="2"/>
+<wire x1="892.81" y1="176.53" x2="892.81" y2="154.94" width="0.1524" layer="91"/>
+</segment>
+</net>
+<net name="OE_PIN" class="0">
 <segment>
 <pinref part="IC4" gate="G$1" pin="OE"/>
@@
 <wire x1="562.61" y1="406.4" x2="562.61" y2="403.86" width="0.1524" layer="91"/>
 <pinref part="R3" gate="G$1" pin="2"/>
+<wire x1="562.61" y1="406.4" x2="562.61" y2="417.83" width="0.1524" layer="91"/>
+<junction x="562.61" y="406.4"/>
+<label x="552.45" y="417.83" size="1.778" layer="95"/>
+</segment>
+<segment>
+<wire x1="914.4" y1="133.35" x2="872.49" y2="133.35" width="0.1524" layer="91"/>
+<pinref part="IC1" gate="G$1" pin="ADC7"/>
+<label x="872.49" y="133.35" size="1.778" layer="95"/>
 </segment>
 </net>
@@
 <wire x1="194.31" y1="735.33" x2="194.31" y2="721.36" width="0.1524" layer="91"/>
 <junction x="194.31" y="721.36"/>
+<label x="102.87" y="698.5" size="1.778" layer="95" rot="R90"/>
 </segment>
 <segment>
@@
 </segment>
 </net>
+<net name="N$7" class="0">
+<segment>
+<pinref part="IC1" gate="G$1" pin="ADC6"/>
+<wire x1="914.4" y1="135.89" x2="892.81" y2="135.89" width="0.1524" layer="91"/>
+<wire x1="892.81" y1="135.89" x2="886.46" y2="135.89" width="0.1524" layer="91"/>
+<wire x1="886.46" y1="135.89" x2="886.46" y2="139.7" width="0.1524" layer="91"/>
+<wire x1="886.46" y1="139.7" x2="886.46" y2="142.24" width="0.1524" layer="91"/>
+<wire x1="886.46" y1="142.24" x2="882.65" y2="142.24" width="0.1524" layer="91"/>
+<wire x1="882.65" y1="139.7" x2="886.46" y2="139.7" width="0.1524" layer="91"/>
+<junction x="886.46" y="139.7"/>
+<pinref part="R41" gate="G$1" pin="1"/>
+<wire x1="892.81" y1="147.32" x2="892.81" y2="135.89" width="0.1524" layer="91"/>
+<junction x="892.81" y="135.89"/>
+<pinref part="SW1" gate="G$1" pin="3"/>
+<pinref part="SW1" gate="G$1" pin="4"/>
+</segment>
+</net>

Commit message: #612 JetRacer ロゴ変更裏、配線間隔修正
Other:
- note added: "2021/10/28 Rev 2.0.14 ボディ装着のため、基板レイアウト変更,RC電源のみで走行可能、プロポマルチ対応,RC GND共通化"
- note added: "RC +B"
- note removed: "2021/9/8 Rev 2.0.14 ボディ装着のため、基板レイアウト変更,RC電源のみで走行可能"
Changed lines of the file:
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@@
 <text x="707.39" y="689.61" size="1.778" layer="94">SN74LVC1G17</text>
 <text x="1085.85" y="684.53" size="1.778" layer="94">SN74LVC1G17</text>
-<text x="826.77" y="485.14" size="6.4516" layer="94">2021/9/8 Rev 2.0.14 ボディ装着のため、基板レイアウト変更,RC電源のみで走行可能</text>
+<text x="788.67" y="469.9" size="3.175" layer="94">2021/10/28 Rev 2.0.14 ボディ装着のため、基板レイアウト変更,RC電源のみで走行可能、プロポマルチ対応,RC GND共通化</text>
 <text x="241.3" y="758.19" size="2.54" layer="97">Analog 3V3</text>
 <text x="38.1" y="599.44" size="3.81" layer="94">受信機から入力</text>
@@
 <text x="693.42" y="115.57" size="3.81" layer="94">ESC</text>
 <text x="693.42" y="134.62" size="3.81" layer="94">サーボ</text>
+<wire x1="96.52" y1="642.62" x2="96.52" y2="623.57" width="0.1524" layer="94"/>
+<wire x1="96.52" y1="642.62" x2="95.25" y2="638.81" width="0.1524" layer="94"/>
+<wire x1="96.52" y1="642.62" x2="97.79" y2="638.81" width="0.1524" layer="94"/>
+<text x="77.47" y="629.92" size="3.81" layer="94">RC +B</text>
+<wire x1="490.22" y1="642.62" x2="490.22" y2="623.57" width="0.1524" layer="94"/>
+<wire x1="490.22" y1="642.62" x2="488.95" y2="638.81" width="0.1524" layer="94"/>
+<wire x1="490.22" y1="642.62" x2="491.49" y2="638.81" width="0.1524" layer="94"/>
+<text x="471.17" y="629.92" size="3.81" layer="94">RC +B</text>
+<wire x1="868.68" y1="637.54" x2="868.68" y2="618.49" width="0.1524" layer="94"/>
+<wire x1="868.68" y1="637.54" x2="867.41" y2="633.73" width="0.1524" layer="94"/>
+<wire x1="868.68" y1="637.54" x2="869.95" y2="633.73" width="0.1524" layer="94"/>
+<text x="849.63" y="624.84" size="3.81" layer="94">RC +B</text>
 </plain>
 <instances>
