File: 0612_jetracer/PCB/612_jetracer_328_020028.sch (EAGLE design)
At the start: 110 parts, among them IC2 JETSON_NANO_NOBORDER, IC3 MULTIPLEXERSMC74HC157A, IC4 PCA9685_BOTTOM, Q1 MOSFET-N_FDN335N, Q2 MOSFET-N_FDN335N, Q3 MOSFET-N_FDN335N, Q4 MOSFET-N_FDN335N, Q5 MOSFET-N_FDN335N, SW1 IS-2245S-G, T5 SN74LVC2G04, T6 SN74LVC2G04, U1 TLP2361, U10 TLP2361, U11 TLP2361, U7 TLP291A, U8 TLP2361, U9 TLP2361, X2 16MHz

Commit message: #612 JetRacer Rev2.0.28 定数の変更　ゲート抵抗４７１に変更。リセット信号コンデンサなし、３２８Pの１０６のコンデンサなし。
Parts:
- C10: value 0.01uF -> DNP
- C6: value 10uF -> DNP
- R1: value 0 -> DNP
- R34, R35, R8: value 10 -> 470
Other:
- note added: "CRISTAL OSCILLATOR"
- note removed: "CRISTAL OSCILLATOR(OPTION)"
- note removed: "水晶発振を取り付けた場合は、取り付けなし"
Changed lines of the file:
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@@
 <part name="R30" library="FaBo-Resistors" deviceset="RESISTOR" device="-0603" value="180"/>
 <part name="GND15" library="FaBo-etc" deviceset="GND" device=""/>
-<part name="R1" library="FaBo-Resistors" deviceset="RESISTOR" device="-0603" value="0"/>
+<part name="R1" library="FaBo-Resistors" deviceset="RESISTOR" device="-0603" value="DNP"/>
 <part name="R3" library="FaBo-Resistors" deviceset="RESISTOR" device="-0603" value="0"/>
 <part name="X_4" library="ngspice-simulation" library_urn="urn:adsk.eagle:library:527439" deviceset="GND" device=""/>
@@
 <part name="U$1" library="FaBo-PIN" deviceset="RC_17PIN_OUTIN" device=""/>
 <part name="X_18" library="ngspice-simulation" library_urn="urn:adsk.eagle:library:527439" deviceset="GND" device=""/>
-<part name="C6" library="FaBo-Capacitor" deviceset="CAPACITOR" device="-0603" value="10uF"/>
+<part name="C6" library="FaBo-Capacitor" deviceset="CAPACITOR" device="-0603" value="DNP"/>
 <part name="C7" library="FaBo-Capacitor" deviceset="CAPACITOR" device="-0402" value="0.1uF"/>
 <part name="R28" library="FaBo-Resistors" deviceset="RESISTOR" device="-0402" value="4.7K/0402"/>
@@
 <part name="X_13" library="ngspice-simulation" library_urn="urn:adsk.eagle:library:527439" deviceset="GND" device=""/>
 <part name="R6" library="FaBo-Resistors" deviceset="RESISTOR" device="-0603" value="330"/>
-<part name="R8" library="FaBo-Resistors" deviceset="RESISTOR" device="-0603" value="10"/>
+<part name="R8" library="FaBo-Resistors" deviceset="RESISTOR" device="-0603" value="470"/>
 <part name="R24" library="FaBo-Resistors" deviceset="RESISTOR" device="-0603" value="100K"/>
 <part name="X_15" library="ngspice-simulation" library_urn="urn:adsk.eagle:library:527439" deviceset="GND" device=""/>
@@
 <part name="X_16" library="ngspice-simulation" library_urn="urn:adsk.eagle:library:527439" deviceset="GND" device=""/>
 <part name="X_17" library="ngspice-simulation" library_urn="urn:adsk.eagle:library:527439" deviceset="GND" device=""/>
-<part name="R34" library="FaBo-Resistors" deviceset="RESISTOR" device="-0603" value="10"/>
-<part name="R35" library="FaBo-Resistors" deviceset="RESISTOR" device="-0603" value="10"/>
+<part name="R34" library="FaBo-Resistors" deviceset="RESISTOR" device="-0603" value="470"/>
+<part name="R35" library="FaBo-Resistors" deviceset="RESISTOR" device="-0603" value="470"/>
 <part name="C5" library="FaBo-Capacitor" deviceset="CAPACITOR" device="-0402" value="0.1uF"/>
 <part name="GND26" library="FaBo-Supply" deviceset="GND" device=""/>
@@
 <part name="SPI-LED" library="FaBo-Connetor" deviceset="FABO-SPI-LED" device=""/>
 <part name="I2C" library="FaBo-Connetor" deviceset="FABO-I2C" device=""/>
-<part name="C10" library="FaBo-Capacitor" deviceset="CAPACITOR" device="-0402" value="0.01uF"/>
+<part name="C10" library="FaBo-Capacitor" deviceset="CAPACITOR" device="-0402" value="DNP"/>
 <part name="GND20" library="FaBo-Supply" deviceset="GND" device=""/>
 </parts>
@@
 <wire x1="411.48" y1="355.6" x2="408.94" y2="358.14" width="0.1524" layer="94"/>
 <text x="111.76" y="429.26" size="1.778" layer="94">option</text>
-<wire x1="76.2" y1="466.09" x2="160.02" y2="466.09" width="0.1524" layer="94" style="longdash"/>
-<wire x1="160.02" y1="466.09" x2="160.02" y2="381" width="0.1524" layer="94" style="longdash"/>
-<wire x1="160.02" y1="381" x2="76.2" y2="381" width="0.1524" layer="94" style="longdash"/>
-<wire x1="76.2" y1="381" x2="76.2" y2="466.09" width="0.1524" layer="94" style="longdash"/>
-<text x="77.47" y="467.36" size="1.778" layer="94">CRISTAL OSCILLATOR(OPTION)</text>
+<text x="77.47" y="467.36" size="1.778" layer="94">CRISTAL OSCILLATOR</text>
 <text x="66.04" y="208.28" size="3.81" layer="97">I2C</text>
 <text x="591.82" y="157.48" size="3.81" layer="97" rot="MR0">OUTLET</text>
-<text x="107.95" y="480.06" size="1.778" layer="94">水晶発振を取り付けた場合は、取り付けなし</text>
-<wire x1="106.68" y1="480.06" x2="157.48" y2="480.06" width="0.1524" layer="94"/>
-<wire x1="157.48" y1="480.06" x2="175.26" y2="462.28" width="0.1524" layer="94"/>
-<wire x1="175.26" y1="462.28" x2="175.26" y2="464.82" width="0.1524" layer="94"/>
 </plain>
 <instances>
