File: 0612_jetracer/PCB/612_jetracer_328_020030.sch (EAGLE design)
At the start: 95 parts, among them IC3 MULTIPLEXERSMC74HC157A, IC4 PCA9685_BOTTOM, Q3 MOSFET-N_FDN335N, Q4 MOSFET-N_FDN335N, Q5 MOSFET-N_FDN335N, SW1 IS-2245S-G, U1 TLP291A, U7 TLP291A, X2 16MHz

Commit message: #612 JetRacer Rev2.0.30 リリースアップデート
Parts:
- added LED1: (no value), FaBo-LED:APA102_IPIXEL
Connections:
- net 5V: now also LED1.VCC
- net AVR_MOSI: now also LED1.SDI
- net AVR_SCK: now also LED1.CKI
- net GND: now also LED1.GND
Changed lines of the file:
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@@
 <part name="GND43" library="FaBo-etc" deviceset="GND" device=""/>
 <part name="GND46" library="FaBo-etc" deviceset="GND" device=""/>
+<part name="LED1" library="FaBo-LED" deviceset="APA102" device="_IPIXEL"/>
+<part name="5V2" library="FaBo-Symbol" deviceset="5V" device=""/>
+<part name="GND47" library="FaBo-Symbol" deviceset="GND" device=""/>
 </parts>
 <sheets>
@@
 <attribute name="VALUE" x="232.156" y="256.54" size="1.778" layer="96"/>
 </instance>
+<instance part="LED1" gate="G$1" x="756.92" y="233.68" smashed="yes">
+<attribute name="NAME" x="749.554" y="241.554" size="1.27" layer="95"/>
+<attribute name="VALUE" x="749.554" y="225.552" size="1.27" layer="96" align="top-left"/>
+</instance>
+<instance part="5V2" gate="G$1" x="741.68" y="241.3" smashed="yes">
+<attribute name="VALUE" x="741.68" y="244.348" size="1.778" layer="96" align="bottom-center"/>
+</instance>
+<instance part="GND47" gate="G$1" x="772.16" y="223.52" smashed="yes">
+<attribute name="VALUE" x="772.16" y="220.472" size="1.778" layer="96" align="top-center"/>
+</instance>
 </instances>
 <busses>
@@
 <junction x="234.95" y="323.85"/>
 </segment>
+<segment>
+<pinref part="LED1" gate="G$1" pin="GND"/>
+<pinref part="GND47" gate="G$1" pin="GND"/>
+<wire x1="767.08" y1="228.6" x2="772.16" y2="228.6" width="0.1524" layer="91"/>
+<wire x1="772.16" y1="228.6" x2="772.16" y2="223.52" width="0.1524" layer="91"/>
+</segment>
 </net>
 <net name="SDA" class="0">
@@
 <wire x1="314.96" y1="223.52" x2="314.96" y2="220.98" width="0.1524" layer="91"/>
 </segment>
+<segment>
+<pinref part="LED1" gate="G$1" pin="VCC"/>
+<pinref part="5V2" gate="G$1" pin="5V"/>
+<wire x1="746.76" y1="236.22" x2="741.68" y2="236.22" width="0.1524" layer="91"/>
+<wire x1="741.68" y1="236.22" x2="741.68" y2="241.3" width="0.1524" layer="91"/>
+</segment>
 </net>
 <net name="RCH1" class="0">
@@
 </segment>
 <segment>
-<wire x1="749.3" y1="276.86" x2="749.3" y2="287.02" width="0.1524" layer="91"/>
+<wire x1="749.3" y1="276.86" x2="749.3" y2="281.94" width="0.1524" layer="91"/>
 <label x="749.3" y="287.02" size="1.778" layer="95" rot="R90"/>
 <pinref part="SPI-LED" gate="G$1" pin="DI"/>
+<pinref part="LED1" gate="G$1" pin="SDI"/>
+<wire x1="749.3" y1="281.94" x2="749.3" y2="287.02" width="0.1524" layer="91"/>
+<wire x1="746.76" y1="233.68" x2="734.06" y2="233.68" width="0.1524" layer="91"/>
+<wire x1="734.06" y1="233.68" x2="734.06" y2="281.94" width="0.1524" layer="91"/>
+<wire x1="734.06" y1="281.94" x2="749.3" y2="281.94" width="0.1524" layer="91"/>
+<junction x="749.3" y="281.94"/>
 </segment>
 </net>
@@
 </segment>
 <segment>
-<wire x1="754.38" y1="276.86" x2="754.38" y2="287.02" width="0.1524" layer="91"/>
+<wire x1="754.38" y1="276.86" x2="754.38" y2="279.4" width="0.1524" layer="91"/>
 <label x="754.38" y="287.02" size="1.778" layer="95" rot="R90"/>
 <pinref part="SPI-LED" gate="G$1" pin="CI"/>
+<wire x1="754.38" y1="279.4" x2="754.38" y2="287.02" width="0.1524" layer="91"/>
+<wire x1="754.38" y1="279.4" x2="739.14" y2="279.4" width="0.1524" layer="91"/>
+<junction x="754.38" y="279.4"/>
+<wire x1="739.14" y1="279.4" x2="739.14" y2="231.14" width="0.1524" layer="91"/>
+<pinref part="LED1" gate="G$1" pin="CKI"/>
+<wire x1="739.14" y1="231.14" x2="746.76" y2="231.14" width="0.1524" layer="91"/>
 </segment>
 </net>
@@
 </sheet>
 </sheets>
-<errors>
-</errors>
 </schematic>
 </drawing>
