File: 0408_jetracer_ledappendboard/PCB/408_jetracer_ledappend_board.sch (EAGLE design)
At the start: 82 parts, among them IC2 SAMD21G18A-AUT, SW1 TS-06104, Y4 32,768Khz_SMD

Commit message: #408 Jetracer_ledappendboardボードデータの追加未完成
Parts:
- removed J1, J2: (no value), FaBo-Template:FABO_BRICK_2PIN
- removed SPI1: FABO-SPI-7PIN, FaBo-Connetor:FABO-SPI-7PIN
- added BAT3, LTS1, LTS2, LTS3: S2B-PH-SM4_TB, FaBo-Connetor:S2B-PH-SM4_TB
- added TR4, TR5: 2N7002, Transistors:1612_2N7002LT1G
- added U$15: FABO-7PINMULTI_SPI, FaBo-Connetor:FABO-7PINMULTI_SPI
- renumbered U$10 to LT4, U$11 to T4, U$12 to T5, U$13 to T6, U$2 to LT1, U$4 to LT2, U$5 to T1, U$6 to T2, U$7 to T3, U$8 to LT3
Connections:
- new net N$35: LTS3.2, TR4.D
- new net N$36: BAT3.2, TR5.D
- net +5V: now also BAT3.1, LTS1.1, LTS2.1, LTS3.1, U$15.5V; no longer J1.VCC, J2.VCC, SPI1.2:5V
- net DGI_GPIO1: now also TR5.G
- net GND: now also TR4.S, TR5.S, U$15.GND; no longer SPI1.1:GND
- net MISO: now also U$15.MISO
- net MOSI: now also U$15.MOSI; no longer SPI1.6:MOSI
- net N$33: now also LTS1.2; no longer J2.GND
- net N$34: now also LTS2.2; no longer J1.GND
- net PA20_TCC0-W6: now also TR4.G
- net SCK: now also U$15.SCK; no longer SPI1.5:SCLK
- net SS: now also U$15.CS

Commit message: #408 JetRacer LED AppendBoard 試作品
Parts:
- removed AD: FH254-106DF08500V, Connettori:1682_20TW-535_STD
- removed BAT3, LTS3: S2B-PH-SM4_TB, FaBo-Connetor:S2B-PH-SM4_TB
- removed C4: 100nF, Condensatori:0015_100NF_0603
- removed C5: 4u7, Condensatori:0474_TAJA475M016RNJ
- removed IOH: FH254-110DF08500V, Connettori:1684_20TW-537
- removed IOL, POWER: FH254-108DF08500V, Connettori:1683_20TW-536
- removed LED1, LED2, LED3: Yellow, Opto:0044_KPT-2012YC
- removed LED4: Green, Opto:0043_KPT-2012SGC
- removed LOGO1: (no value), FaBo-Logo:LOGO_OSHW-M_BOTTOM
- removed R15, R24, R25, R4, R6, R7: 470, FaBo-Resistors:RESISTOR-0603
- removed R26, R27, R28, R29, R30, R31, R32, R33, R34: 220, FaBo-Resistors:RESISTOR-0603
- removed T1, T2, T3, T4, T5, T6: T2N7002AK, FaBo-Mosfet:T2N7002AK
- removed TR4, TR5: 2N7002, Transistors:1612_2N7002LT1G
- added P1: (no value), FaBo-Connetor:4PIN_HEADER_1.25MM
- added R1: 470/0806, FaBo-Resistors:RESISTOR-0805
- added TR10, TR11, TR12, TR13, TR14, TR15, TR16, TR6, TR7, TR8, TR9: 2N7002, Transistors:1612_2N7002LT1G
- LTS1, LTS2: value S2B-PH-SM4_TB -> (none); device FaBo-Connetor:S2B-PH-SM4_TB -> FaBo-Connetor:B2B-XH-AM
- R10, R11, R12, R13, R14, R16, R20, R21, R22, R23: value 470 -> 470/0806; device FaBo-Resistors:RESISTOR-0603 -> FaBo-Resistors:RESISTOR-0805
- R17, R18, R19: value 220 -> 470/0806; device FaBo-Resistors:RESISTOR-0603 -> FaBo-Resistors:RESISTOR-0805
- renumbered U$15 to SPI
Connections:
- removed net N$29: R26.1, R32.1, T4.1:GATE
- removed net N$30: R27.1, R33.1, T5.1:GATE
- removed net N$35: LTS3.2, TR4.D
- removed net N$36: BAT3.2, TR5.D
- removed net N$4: LED4.C, R15.2
- removed net N$56: POWER.1
- removed net PWRIN: POWER.8
- net +3V3: no longer LED1.A, LED2.A, LED3.A, LED4.A, POWER.2, POWER.4
- net +5V: now also P1.2, R22.2, R23.2; no longer BAT3.1, LTS1.1, LTS2.1, LTS3.1, POWER.5
- net DGI_GPIO0: now also TR7.G
- net DGI_GPIO1: no longer IOL.8, TR5.G
- net DGI_GPIO2: no longer IOH.1
- net DGI_GPIO3: no longer IOH.2
- net GND: now also P1.1, TR10.S, TR11.S, TR12.S, TR13.S, TR14.S, TR15.S, TR16.S, TR6.S, TR7.S, TR8.S, TR9.S; no longer C4.2, C5.-, IOH.7, POWER.6, POWER.7, R15.1, R29.2, R30.2, R31.2, R32.2, R33.2, R34.2, T1.2:SOURCE, T2.2:SOURCE, T3.2:SOURCE, T4.2:SOURCE, T5.2:SOURCE, T6.2:SOURCE, TR4.S, TR5.S
- net MISO: no longer IOH.5
- net MOSI: no longer IOH.4
- net N$1: now also R13.1, TR9.D; no longer LED1.C, R4.2
- net N$11: now also R11.2; no longer R10.2
- net N$12: now also R12.2; no longer R16.2
- net N$13: now also R13.2; no longer R14.2
- net N$14: now also R14.2; no longer R13.2
- net N$15: now also R14.1, TR10.D; no longer R10.1, R13.1, T3.3:DRAIN
- net N$16: now also R17.1, TR12.D; no longer R11.1, R14.1, T2.3:DRAIN
- net N$17: now also R16.1, TR11.D; no longer R17.1, R29.1, T1.1:GATE
- net N$18: now also LTS1.2, R22.1; no longer R18.1, R30.1, T2.1:GATE
- net N$19: now also LTS2.2, R23.1; no longer R19.1, R31.1, T3.1:GATE
- net N$2: now also R10.1, TR6.D; no longer LED2.C, R6.2
- net N$20: now also R16.2; no longer R22.2
- net N$21: now also R17.2; no longer R21.2
- net N$22: now also R18.2; no longer R20.2
- net N$23: now also R19.2; no longer R25.2
- net N$24: now also R20.2; no longer R24.2
- net N$25: now also R21.2; no longer R23.2
- net N$26: now also R18.1, TR13.D; no longer R22.1, R25.1, T4.3:DRAIN
- net N$27: now also R20.1, TR15.D; no longer R21.1, R24.1, T5.3:DRAIN
- net N$28: now also R19.1, TR14.D; no longer R20.1, R23.1, T6.3:DRAIN
- net N$3: now also R1.1, TR3.D; no longer LED3.C, R7.2
- net N$31: now also R21.1, TR16.D; no longer R28.1, R34.1, T6.1:GATE
- net N$33: now also LTS1.1; no longer LTS1.2
- net N$34: now also LTS2.1; no longer LTS2.2
- net N$5: now also R11.1, TR7.D; no longer R7.1, TR3.D
- net N$6: now also R1.2; no longer R12.2
- net N$8: now also TR8.D; no longer R16.1, T1.3:DRAIN
- net N$9: now also R10.2; no longer R11.2
- net PA02_AIN0: no longer AD.1
- net PA03_AREFA: no longer C4.1, C5.+, IOH.8
- net PA04_AIN4: no longer AD.4
- net PA05_AIN5: no longer AD.5
- net PA08_TCC0-W0: no longer IOL.3, R19.2
- net PA09_TCC0-W1: now also TR13.G; no longer IOL.4, R26.2
- net PA10_TCC0-W2: now also TR12.G; no longer IOL.2, R18.2
- net PA11_TCC0-W3: now also TR11.G; no longer IOL.1, R17.2
- net PA14_TCC0-W4: now also TR6.G; no longer IOL.5, R27.2
- net PA15_TCC0-W5: now also TR3.G; no longer IOL.6, R28.2
- net PA20_TCC0-W6: no longer IOL.7, TR4.G
- net PA27_TX_LED: no longer R4.1
- net PB02_AIN10: no longer AD.6
- net PB03_RX_LED: no longer R6.1
- net PB08_AIN2: no longer AD.2
- net PB09_AIN3: no longer AD.3
- net PB10_S4_SPI_MOSI: now also TR10.G
- net PB11_S4_SPI_SCK: now also TR9.G
- net PB12_S4_SPI_MISO: now also TR8.G
- net RESET: no longer POWER.3
- net SCK: no longer IOH.6, TR3.G
- net SCL: now also P1.3; no longer IOH.10
- net SDA: now also P1.4; no longer IOH.9
- net SS: no longer IOH.3
Other:
- note added: "0.0.0"
- note removed: "1.0.1"
- moved on the sheet: CN2, LTS1, LTS2, R10, R11, R12, R13, R14, R16, R17, R18, R19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
